File: e788v01a/LR2021_e788v01a_868_915_eval_module.kicad_pcb (KiCad board)
At the start: 4 copper layers, 86 x 56 mm, 156 parts, among them J1_DISP Header 8, J2_DISP Header 10, J3_DISP Header 8, J4_DISP Header 6, J5 GROVE-CONNECTOR-DIP-320110034, J6 GROVE-CONNECTOR-DIP-320110034, J7_SWD HEADER-2X4P-2.54-SMD, K1_USER TS-1111A, K2_RESET TS-1111A, Q1 Xtal, U1 LR20xx, U2 Seeeduino XIAO nRF, U3 ZJY-2864KSWPG01, U4 NCP59800BMNADJTAG

Commit message: Fixed warnings
Parts:
- Logo ESD1: renamed from Logo ESD
- Logo Recycling1: renamed from Logo Recycling
- renumbered 868M to 868M1, 915M to 915M1, ANT_HF to ANT_HF1, ANT_LF to ANT_LF1, IDCC to IDCC1, J1_DISP to J1_DISP1, J2_DISP to J2_DISP1, J3_DISP to J3_DISP1, J4_DISP to J4_DISP1, J7_SWD to J7_SWD1, K1_USER to K1_USER1, K2_RESET to K2_RESET1, Other to Other1, R4_N to R4_N1, Shield to Shield1
Connections:
- J1_DISP1 pad 1: (no net) -> unconnected-(J1_DISP1-D0-Pad1)
- J1_DISP1 pad 2: (no net) -> unconnected-(J1_DISP1-D1-Pad2)
- J1_DISP1 pad 4: (no net) -> unconnected-(J1_DISP1-D3-Pad4)
- J1_DISP1 pad 5: (no net) -> unconnected-(J1_DISP1-D4-Pad5)
- J1_DISP1 pad 6: (no net) -> unconnected-(J1_DISP1-D5-Pad6)
- J1_DISP1 pad 7: (no net) -> unconnected-(J1_DISP1-D6-Pad7)
- J1_DISP1 pad 8: (no net) -> unconnected-(J1_DISP1-D7-Pad8)
- J2_DISP1 pad 1: (no net) -> unconnected-(J2_DISP1-D8-Pad1)
- J2_DISP1 pad 8: (no net) -> unconnected-(J2_DISP1-AVDD-Pad8)
- J3_DISP1 pad 1: (no net) -> unconnected-(J3_DISP1-NC-Pad1)
- J3_DISP1 pad 2: (no net) -> unconnected-(J3_DISP1-IOREF-Pad2)
- J3_DISP1 pad 4: (no net) -> unconnected-(J3_DISP1-+3V3-Pad4)
- J3_DISP1 pad 8: (no net) -> unconnected-(J3_DISP1-VIN-Pad8)
- J4_DISP1 pad 1: (no net) -> unconnected-(J4_DISP1-A0-Pad1)
- J4_DISP1 pad 2: (no net) -> unconnected-(J4_DISP1-A1-Pad2)
- J4_DISP1 pad 3: (no net) -> unconnected-(J4_DISP1-A2-Pad3)
- J4_DISP1 pad 4: (no net) -> unconnected-(J4_DISP1-A3-Pad4)
- J4_DISP1 pad 5: (no net) -> unconnected-(J4_DISP1-A4-Pad5)
- J4_DISP1 pad 6: (no net) -> unconnected-(J4_DISP1-A5-Pad6)
- JH2 pad 8: (no net) -> unconnected-(JH2-AVDD-Pad8)
- JH3 pad 1: (no net) -> unconnected-(JH3-NC-Pad1)
- JH3 pad 2: (no net) -> unconnected-(JH3-IOREF-Pad2)
- JH3 pad 8: (no net) -> unconnected-(JH3-VIN-Pad8)
- JH4 pad 3: (no net) -> unconnected-(JH4-A2-Pad3)
- JH4 pad 5: (no net) -> unconnected-(JH4-A4-Pad5)
- JH4 pad 6: (no net) -> unconnected-(JH4-A5-Pad6)
- U1 pad 18: (no net) -> unconnected-(U1-DIO6-Pad18)
- U1 pad 19: (no net) -> unconnected-(U1-DIO5-Pad19)
- U1 pad 8: (no net) -> unconnected-(U1-DIO10-Pad8)
- U1 pad 9: (no net) -> unconnected-(U1-DIO9-Pad9)
- U2 pad 19: (no net) -> unconnected-(U2-SAMD11_RST-Pad19)
- U2 pad 21: (no net) -> unconnected-(U2-SAMD11_SWDIO-Pad21)
- U2 pad 22: (no net) -> unconnected-(U2-SAMD11_SWCLK-Pad22)
- U2 pad 23: (no net) -> unconnected-(U2-D16-Pad23)
- U2 pad 29: (no net) -> unconnected-(U2-D18-Pad29)
- U2 pad 30: (no net) -> unconnected-(U2-D17-Pad30)
- U3 pad 12: (no net) -> unconnected-(U3-BS2-Pad12)
- U3 pad 16: (no net) -> unconnected-(U3-R/W-Pad16)
- U3 pad 17: (no net) -> unconnected-(U3-E/RD-Pad17)
- U3 pad 21: (no net) -> unconnected-(U3-D3-Pad21)
- U3 pad 22: (no net) -> unconnected-(U3-D4-Pad22)
- U3 pad 23: (no net) -> unconnected-(U3-D5-Pad23)
- U3 pad 24: (no net) -> unconnected-(U3-D6-Pad24)
- U3 pad 25: (no net) -> unconnected-(U3-D7-Pad25)
- U3 pad 7: (no net) -> unconnected-(U3-NC-Pad7)
