File: e788v01a/LR2021_e788v01a_868_915_eval_module.kicad_sch (KiCad schematic)
At the start: 125 parts, among them J1_DISP Header 8, J2_DISP Header 10, J3_DISP Header 8, J4_DISP Header 6, Q1 Xtal, U1 LR20xx, U2 Seeeduino XIAO nRF, U4 NCP59800BMNADJTAG

Commit message: Fixed warnings
Parts:
- Logo ESD1: renamed from Logo ESD
- Logo Recycling1: renamed from Logo Recycling
- renumbered 868M to 868M1, 915M to 915M1, ANT_HF to ANT_HF1, ANT_LF to ANT_LF1, IDCC to IDCC1, J1_DISP to J1_DISP1, J2_DISP to J2_DISP1, J3_DISP to J3_DISP1, J4_DISP to J4_DISP1, Other to Other1, R4_N to R4_N1, Shield to Shield1
Changed lines of the file:
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@@
 		(in_pos_files yes)
 		(dnp no)
-		(property "Reference" "IDCC"
+		(property "Reference" "IDCC1"
 			(at 268.002 160.655 0)
 			(show_name no)
@@
 			(project "LR2021_e788v01a_868_915_eval_module"
 				(path "/4d621f81-96a6-4f9d-9b52-24879b1dad45"
-					(reference "IDCC")
+					(reference "IDCC1")
 					(unit 1)
 				)
@@
 			)
 		)
-		(pin "0"
-		)
 		(instances
 			(project "LR2021_e788v01a_868_915_eval_module"
@@
 		(in_pos_files yes)
 		(dnp no)
-		(property "Reference" "Shield"
+		(property "Reference" "Shield1"
 			(at 533.412 382.983 0)
 			(show_name no)
@@
 			(project "LR2021_e788v01a_868_915_eval_module"
 				(path "/4d621f81-96a6-4f9d-9b52-24879b1dad45"
-					(reference "Shield")
+					(reference "Shield1")
 					(unit 1)
 				)
@@
 		(in_pos_files yes)
 		(dnp no)
-		(property "Reference" "ANT_LF"
+		(property "Reference" "ANT_LF1"
 			(at 463.692 103.82 90)
 			(show_name no)
@@
 			(project "LR2021_e788v01a_868_915_eval_module"
 				(path "/4d621f81-96a6-4f9d-9b52-24879b1dad45"
-					(reference "ANT_LF")
+					(reference "ANT_LF1")
 					(unit 1)
 				)
@@
 		(in_pos_files yes)
 		(dnp no)
-		(property "Reference" "J1_DISP"
+		(property "Reference" "J1_DISP1"
 			(at 213.582 249.301 0)
 			(show_name no)
@@
 			(project "LR2021_e788v01a_868_915_eval_module"
 				(path "/4d621f81-96a6-4f9d-9b52-24879b1dad45"
-					(reference "J1_DISP")
+					(reference "J1_DISP1")
 					(unit 1)
 				)
@@
 		(in_pos_files yes)
 		(dnp no)
-		(property "Reference" "J3_DISP"
+		(property "Reference" "J3_DISP1"
 			(at 250.412 280.543 0)
 			(show_name no)
@@
 			(project "LR2021_e788v01a_868_915_eval_module"
 				(path "/4d621f81-96a6-4f9d-9b52-24879b1dad45"
-					(reference "J3_DISP")
+					(reference "J3_DISP1")
 					(unit 1)
 				)
@@
 		(in_pos_files yes)
 		(dnp no)
-		(property "Reference" "868M"
+		(property "Reference" "868M1"
 			(at 524.892 347.013 0)
 			(show_name no)
@@
 			(project "LR2021_e788v01a_868_915_eval_module"
 				(path "/4d621f81-96a6-4f9d-9b52-24879b1dad45"
-					(reference "868M")
+					(reference "868M1")
 					(unit 1)
 				)
@@
 		(in_pos_files yes)
 		(dnp no)
-		(property "Reference" "Logo ESD"
+		(property "Reference" "Logo ESD1"
 			(at 483.982 383.421 0)
 			(show_name no)
@@
 			)
 		)
-		(pin "0"
-		)
 		(instances
 			(project "LR2021_e788v01a_868_915_eval_module"
 				(path "/4d621f81-96a6-4f9d-9b52-24879b1dad45"
-					(reference "Logo ESD")
+					(reference "Logo ESD1")
 					(unit 1)
 				)
@@
 		(in_pos_files yes)
 		(dnp no)
-		(property "Reference" "J2_DISP"
+		(property "Reference" "J2_DISP1"
 			(at 213.582 278.765 0)
 			(show_name no)
@@
 			(project "LR2021_e788v01a_868_915_eval_module"
 				(path "/4d621f81-96a6-4f9d-9b52-24879b1dad45"
-					(reference "J2_DISP")
+					(reference "J2_DISP1")
 					(unit 1)
 				)
@@
 			)
 		)
-		(pin "0"
-		)
 		(instances
 			(project "LR2021_e788v01a_868_915_eval_module"
@@
 			)
 		)
-		(pin "0"
-		)
 		(instances
 			(project "LR2021_e788v01a_868_915_eval_module"
@@
 		(in_pos_files yes)
 		(dnp no)
-		(property "Reference" "915M"
+		(property "Reference" "915M1"
 			(at 525.392 354.013 0)
 			(show_name no)
@@
 			(project "LR2021_e788v01a_868_915_eval_module"
 				(path "/4d621f81-96a6-4f9d-9b52-24879b1dad45"
-					(reference "915M")
+					(reference "915M1")
 					(unit 1)
 				)
@@
 		(in_pos_files yes)
 		(dnp no)
-		(property "Reference" "Other"
+		(property "Reference" "Other1"
 			(at 525.392 361.013 0)
 			(show_name no)
@@
 			(project "LR2021_e788v01a_868_915_eval_module"
 				(path "/4d621f81-96a6-4f9d-9b52-24879b1dad45"
-					(reference "Other")
+					(reference "Other1")
 					(unit 1)
 				)
@@
 		(in_pos_files yes)
 		(dnp no)
-		(property "Reference" "Logo Recycling"
+		(property "Reference" "Logo Recycling1"
 			(at 483.982 386.421 0)
 			(show_name no)
@@
 			)
 		)
-		(pin "0"
-		)
 		(instances
 			(project "LR2021_e788v01a_868_915_eval_module"
 				(path "/4d621f81-96a6-4f9d-9b52-24879b1dad45"
-					(reference "Logo Recycling")
+					(reference "Logo Recycling1")
 					(unit 1)
 				)
@@
 		(in_pos_files yes)
 		(dnp no)
-		(property "Reference" "R4_N"
+		(property "Reference" "R4_N1"
 			(at 335.996 259.734 90)
 			(show_name no)
@@
 			(project "LR2021_e788v01a_868_915_eval_module"
 				(path "/4d621f81-96a6-4f9d-9b52-24879b1dad45"
-					(reference "R4_N")
+					(reference "R4_N1")
 					(unit 1)
 				)
@@
 		(in_pos_files yes)
 		(dnp no)
-		(property "Reference" "J4_DISP"
+		(property "Reference" "J4_DISP1"
 			(at 250.988 249.301 0)
 			(show_name no)
@@
 			(project "LR2021_e788v01a_868_915_eval_module"
 				(path "/4d621f81-96a6-4f9d-9b52-24879b1dad45"
-					(reference "J4_DISP")
+					(reference "J4_DISP1")
 					(unit 1)
 				)
@@
 			)
 		)
-		(pin "0"
-		)
 		(instances
 			(project "LR2021_e788v01a_868_915_eval_module"
@@
 		(in_pos_files yes)
 		(dnp no)
-		(property "Reference" "ANT_HF"
+		(property "Reference" "ANT_HF1"
 			(at 402.192 103.82 90)
 			(show_name no)
@@
 			(project "LR2021_e788v01a_868_915_eval_module"
 				(path "/4d621f81-96a6-4f9d-9b52-24879b1dad45"
-					(reference "ANT_HF")
+					(reference "ANT_HF1")
 					(unit 1)
 				)
