File: e788v01a/LR2021_e788v01a_868_915_eval_module_accessories.kicad_sch (KiCad schematic)
At the start: 31 parts, among them J5 GROVE-CONNECTOR-DIP-320110034, J6 GROVE-CONNECTOR-DIP-320110034, J7_SWD HEADER-2X4P-2.54-SMD, K1_USER TS-1111A, K2_RESET TS-1111A, U3 ZJY-2864KSWPG01

Commit message: Fixed warnings
Parts:
- renumbered J7_SWD to J7_SWD1, K1_USER to K1_USER1, K2_RESET to K2_RESET1
Changed lines of the file:
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@@
 		(in_pos_files yes)
 		(dnp no)
-		(property "Reference" "K2_RESET"
+		(property "Reference" "K2_RESET1"
 			(at 140 339.489 0)
 			(show_name no)
@@
 			(project "LR2021_e788v01a_868_915_eval_module"
 				(path "/4d621f81-96a6-4f9d-9b52-24879b1dad45/52a010f0-de47-46b4-9541-17dcb44a4527"
-					(reference "K2_RESET")
+					(reference "K2_RESET1")
 					(unit 1)
 				)
@@
 		(in_pos_files yes)
 		(dnp no)
-		(property "Reference" "K1_USER"
+		(property "Reference" "K1_USER1"
 			(at 140 316.489 0)
 			(show_name no)
@@
 			(project "LR2021_e788v01a_868_915_eval_module"
 				(path "/4d621f81-96a6-4f9d-9b52-24879b1dad45/52a010f0-de47-46b4-9541-17dcb44a4527"
-					(reference "K1_USER")
+					(reference "K1_USER1")
 					(unit 1)
 				)
@@
 		(in_pos_files yes)
 		(dnp no)
-		(property "Reference" "J7_SWD"
+		(property "Reference" "J7_SWD1"
 			(at 139.75 136.95 0)
 			(show_name no)
@@
 			(project "LR2021_e788v01a_868_915_eval_module"
 				(path "/4d621f81-96a6-4f9d-9b52-24879b1dad45/52a010f0-de47-46b4-9541-17dcb44a4527"
-					(reference "J7_SWD")
+					(reference "J7_SWD1")
 					(unit 1)
 				)
